File: V1/B-CAN-giraffe_v1.brd (EAGLE design)
At the start: 100.3 x 31.8 mm, 7 parts, among them J3 OBDII-FEMALE-CUT, J4 VERT_RJ45, SW1 4XDPSTSMT

Commit message: Push V2 and organize into folders
Parts:
- added J5: VERT_RJ45, comma.ai:GLX-S-88M
- moved J3 14.0 mm to (91.4, 9.53)
Connections:
- net CAN1_H: now also J4.6, SW1.1
- net CAN1_L: now also J4.3, SW1.2
- net CAN3_H: now also J5.6; no longer J4.6
- net CAN3_L: now also J5.3; no longer J4.3
Routing:
- net CAN3_H: track 59.8 -> 0.00 mm, vias 2 -> 0
- net CAN3_L: track 55.7 -> 0.04 mm, vias 2 -> 0
- net CAN2_L: track 129.9 -> 84.0 mm, vias 4 -> 3
- net CAN1_L: track 91.1 -> 60.7 mm
- net K_LIN: track 111.5 -> 82.6 mm
- net 12VIN: track 65.7 -> 79.7 mm
- net IGN: track 64.5 -> 51.7 mm, vias 5 -> 4
- net CAN1_H: track 66.5 -> 77.9 mm, vias 0 -> 1
- net CAN2_H: track 118.1 -> 112.9 mm, vias 4 -> 3
- net L_LIN: track 85.3 -> 82.2 mm
- net GND: vias 5 -> 4
Other:
- board size 100.3 x 31.8 mm -> 113 x 31.8 mm
- board text added: "8/8/17"
- board text added: "vanillagorillaa"
- board text removed: "11/3/17"
