File: B-CAN_Board.sch (EAGLE design)
At the start: 3 parts, among them X1 GLX-S-88M

Commit message: God this used to look so ugly, lets make it nice
Parts:
- removed U$1: 670-2297-ND, 670-2297-ND:670-2297-ND
- removed U$2: 670-2910-ND, 670-2910-ND:670-2910-ND
- removed X1: GLX-S-88M, con-kycon:GLX-S-88M
- added J1: RA-RJ45RA, comma.ai:RA-RJ45RA
- added J2, J3: MX34032UF2, MX34032UF2:MX34032UF2
Connections:
- removed net N$1: U$1.SOL_IN, U$2.SOL_IN
- removed net N$10: U$1.BUS-DATA, U$2.BUS-DATA
- removed net N$11: U$1.SOL_OUT, U$2.SOL_OUT
- removed net N$2: U$1.B-CAN_L, U$2.B-CAN_L, X1.3
- removed net N$3: U$1.TAM, U$2.TAM
- removed net N$4: U$1.SENSOR_COM, U$2.SENSOR_COM
- removed net N$5: U$1.IG2_A/C, U$2.IG2_A/C
- removed net N$6: U$1.RR_DEF_RLY_CL-, U$2.RR_DEF_RLY_CL-
- removed net N$7: U$1.B-CAN_H, U$2.B-CAN_H, X1.6
- removed net N$8: U$1.TR, U$2.TR
- removed net N$9: U$1.GND, U$2.GND, X1.5
- new net B-CAN_H: J1.6, J2.P25, J3.P25
- new net B-CAN_L: J1.3, J2.P8, J3.P8
- new net BUS-DATA: J2.P29, J3.P29
- new net GND: J2.P28, J3.P28
- new net IG2_A/C: J2.P32, J3.P32
- new net RR_DEF_RLY_CL-: J2.P21, J3.P21
- new net SENSOR_COM: J2.P12, J3.P12
- new net SOL_IN: J2.P14, J3.P14
- new net SOL_OUT: J2.P30, J3.P30
- new net TAM: J2.P11, J3.P11
- new net TR: J2.P27, J3.P27
